File: hardware/esp32c3-wifi-dev/esp32c3-wifi-dev.kicad_pcb (KiCad board)
At the start: 2 copper layers, 79.5 x 31.5 mm, 14 parts, among them J1 Conn_01x02, J2 Conn_01x04, J3 Conn_01x04, U1 xiao-rp2040

Commit message: Add order version
Parts:
- moved G*** 1.00 mm to (201.0, 65.5)
Connections:
- U1 pad 3: unconnected-(U1-P28_A2_D2-Pad3) -> /RP2040-TXD
- U1 pad 4: /RP2040-CSn -> /RP2040-RXD
- U1 pad 7: /RP2040-TXD -> unconnected-(U1-P0_TX_D6-Pad7)
- U1 pad 8: /RP2040-RXD -> /RP2040-CSn
Routing:
- net /RP2040-RXD: track 42.2 -> 31.6 mm
- net /ESP32C3-SCK: track 36.4 -> 29.2 mm
- net /ESP32C3-MISO: track 38.0 -> 30.9 mm
- net /RP2040-TXD: track 26.9 -> 33.3 mm
- net /ESP32C3-MOSI: track 39.6 -> 34.1 mm
- net /RP2040-CSn: track 16.8 -> 13.1 mm, vias 0 -> 1
Other:
- board text added: "MnemOS WiFi Development Jig July 2023 UART + SPI Host Adapter onevariable.com"
- board text removed: "MnemOS WiFi Development Jig July 2023 UART + SPI Host Adapter"
