File: hardware/esp32c3-wifi-dev/esp32c3-wifi-dev.kicad_sch (KiCad schematic)
At the start: 13 parts, among them J1 Conn_01x02, J2 Conn_01x04, J3 Conn_01x04, U1 xiao-rp2040

Commit message: Add order version
Connections:
- net RP2040-CSn: now also U1.8 (P1_RX_D7); no longer U1.4 (P29_A3_D3)
- net RP2040-RXD: now also U1.4 (P29_A3_D3); no longer U1.8 (P1_RX_D7)
- net RP2040-TXD: now also U1.3 (P28_A2_D2); no longer U1.7 (P0_TX_D6)
Changed lines of the file:
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@@
     (effects (font (size 1.27 1.27)) (justify left bottom))
   )
-  (label "RP2040-CSn" (at 80.01 80.01 180) (fields_autoplaced)
-    (effects (font (size 1.27 1.27)) (justify right bottom))
+  (label "RP2040-CSn" (at 120.65 87.63 0) (fields_autoplaced)
+    (effects (font (size 1.27 1.27)) (justify left bottom))
   )
   (label "RP2040-D1" (at 142.24 153.67 180) (fields_autoplaced)
@@
     (effects (font (size 1.27 1.27)) (justify left bottom))
   )
-  (label "RP2040-TXD" (at 80.01 87.63 180) (fields_autoplaced)
+  (label "RP2040-TXD" (at 80.01 77.47 180) (fields_autoplaced)
     (effects (font (size 1.27 1.27)) (justify right bottom))
   )
@@
     (effects (font (size 1.27 1.27)) (justify right bottom))
   )
-  (label "RP2040-RXD" (at 120.65 87.63 0) (fields_autoplaced)
-    (effects (font (size 1.27 1.27)) (justify left bottom))
+  (label "RP2040-RXD" (at 80.01 80.01 180) (fields_autoplaced)
+    (effects (font (size 1.27 1.27)) (justify right bottom))
   )
   (label "ESP32C3-CSn" (at 166.37 80.01 180) (fields_autoplaced)
